File: KiCad schem/ELECTRIC LIGHTER.kicad_sch (KiCad schematic)
At the start: 5 parts, among them SW1 Button, U1 TP4056

Commit message: Add files via upload
Parts:
- 3.7V1: symbol Device:Battery_Cell -> EL library:Battery_Cell
- R1: symbol Device:Heater -> EL library:Heater
- SW1: symbol Switch:SW_Push -> EL library:SW_Push
- U1: symbol Battery_Management:TP4056-42-ESOP8 -> EL library:TP4056-42-ESOP8
- USBC1: symbol Connector:USB_C_Receptacle_PowerOnly_6P -> EL library:USB_C_Receptacle_PowerOnly_6P
Connections:
- net at R1.1: now also 3.7V1.2 (-), U1.9 (B-); no longer U1.2 (OUT+)
- net at 3.7V1.1 (+), U1.3 (B+): now also SW1.2
- net at U1.2 (OUT+): no longer SW1.2
- new net: U1.5 (IN+), USBC1. (-)
Changed lines of the file:
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@@
 	(generator_version "9.0")
 	(paper "A4")
-	(wire
-		(pts
-			(xy 152.4 100.33) (xy 152.4 132.08)
+	(junction
+		(at 144.78 102.87)
+		(diameter 0)
+		(color 0 0 0 0)
+	)
+	(junction
+		(at 147.32 102.87)
+		(diameter 0)
+		(color 0 0 0 0)
+	)
+	(wire
+		(pts
+			(xy 144.78 102.87) (xy 144.78 104.14)
+		)
+		(stroke
+			(width 0)
+			(type default)
+		)
+	)
+	(wire
+		(pts
+			(xy 152.4 102.87) (xy 152.4 132.08)
 		)
 		(stroke
@@
 	(wire
 		(pts
-			(xy 139.7 100.33) (xy 139.7 118.11)
-		)
-		(stroke
-			(width 0)
-			(type default)
-		)
-	)
-	(wire
-		(pts
-			(xy 144.78 100.33) (xy 144.78 104.14)
-		)
-		(stroke
-			(width 0)
-			(type default)
-		)
-	)
-	(wire
-		(pts
-			(xy 147.32 100.33) (xy 147.32 104.14)
+			(xy 144.78 100.33) (xy 144.78 102.87)
+		)
+		(stroke
+			(width 0)
+			(type default)
+		)
+	)
+	(wire
+		(pts
+			(xy 139.7 118.11) (xy 139.7 102.87)
+		)
+		(stroke
+			(width 0)
+			(type default)
+		)
+	)
+	(wire
+		(pts
+			(xy 147.32 100.33) (xy 147.32 102.87)
 		)
 		(stroke
@@
 	(wire
 		(pts
+			(xy 147.32 102.87) (xy 147.32 104.14)
+		)
+		(stroke
+			(width 0)
+			(type default)
+		)
+	)
+	(wire
+		(pts
+			(xy 147.32 102.87) (xy 152.4 102.87)
+		)
+		(stroke
+			(width 0)
+			(type default)
+		)
+	)
+	(wire
+		(pts
 			(xy 149.86 109.22) (xy 149.86 104.14)
 		)
@@
 		(pts
 			(xy 140.97 132.08) (xy 139.7 132.08)
+		)
+		(stroke
+			(width 0)
+			(type default)
+		)
+	)
+	(wire
+		(pts
+			(xy 139.7 102.87) (xy 144.78 102.87)
 		)
 		(stroke
@@
 	)
 	(symbol
-		(lib_id "Device:Heater")
+		(lib_id "EL library:Heater")
 		(at 139.7 121.92 0)
 		(unit 1)
@@
 	)
 	(symbol
-		(lib_id "Device:Battery_Cell")
+		(lib_id "EL library:Battery_Cell")
 		(at 144.78 109.22 270)
 		(unit 1)
@@
 	)
 	(symbol
-		(lib_id "Battery_Management:TP4056-42-ESOP8")
+		(lib_name "TP4056-42-ESOP8_1")
+		(lib_id "EL library:TP4056-42-ESOP8")
 		(at 146.05 87.63 0)
 		(unit 1)
@@
 	)
 	(symbol
-		(lib_id "Switch:SW_Push")
+		(lib_id "EL library:SW_Push")
 		(at 146.05 132.08 0)
 		(unit 1)
@@
 	)
 	(symbol
-		(lib_id "Connector:USB_C_Receptacle_PowerOnly_6P")
+		(lib_name "USB_C_Receptacle_PowerOnly_6P_1")
+		(lib_id "EL library:USB_C_Receptacle_PowerOnly_6P")
 		(at 143.51 62.23 270)
 		(unit 1)
